Commit message: udpate

File: urdf/quadcopter.urdf (robot description, URDF)
Before this commit: robot quadcopter, 1 links, 0 joints
Links:
- link base_link: geometry collision mesh filename=package://uav_simulator/urdf/quadcopter/meshes/quadcopter.s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 scale=1.0 1.0 1.0; visual mesh filename=package://uav_simulator/urdf/quadcopter/meshes/quadcopter.d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 scale=1.0 1.0 1.0

Commit message: final model & fix random move issue

File: urdf/quadcopter.urdf (robot description, URDF)
Before this commit: robot quadcopter, 1 links, 0 joints
Links:
- link base_link: geometry collision mesh filename=package://uav_simulator/urdf/quadcopter/meshes/CERLAB_quadc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 scale=1.5 1.5 1.5; visual mesh filename=package://uav_simulator/urdf/quadcopter/meshes/CERLAB_quadc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 scale=1.5 1.5 1.5

Commit message: update PID

File: urdf/quadcopter.urdf (robot description, URDF)
Before this commit: robot quadcopter, 1 links, 0 joints
Links:
- link base_link: mass 1.477 -> 1.54
